Commit message: added ultrasonic

File: apollo_description/urdf/xacro/accessories.urdf.xacro (robot description, xacro)
@@ -69,3 +69,48 @@
     </gazebo>
   </xacro:macro>
+  <xacro:macro name="ultrasonic" params="name xyz rpy">
+    <link name="${name}_ultrasonic"/>
+    <joint name="${name}_us_joint" type="fixed">
+      <parent link="base_link"/>
+      <child link="${name}_ultrasonic"/>
+      <origin xyz="${xyz}" rpy="${rpy}"/>
+    </joint>
+    <gazebo reference="${name}_ultrasonic">
+     <sensor type="ray" name="${name}_ultrasonic_sen">
+        <pose>${xyz} ${rpy}</pose>
+        <update_rate>50</update_rate>
+        <ray>
+           <scan>
+              <horizontal>
+                 <samples>1</samples>
+                 <resolution>1.0</resolution>
+                 <min_angle>-0.1308995</min_angle>
+                 <max_angle>0.1308995</max_angle>
+              </horizontal>
+              <vertical>
+                 <samples>1</samples>
+                 <resolution>1</resolution>
+                 <min_angle>-0.01</min_angle>
+                 <max_angle>0.01</max_angle>
+              </vertical>
+           </scan>
+           <range>
+              <min>0.02</min>
+              <max>4.0</max>
+              <resolution>0.02</resolution>
+           </range>
+        </ray>
+        <plugin filename="libgazebo_ros_range.so" name="gazebo_ros_range">
+           <gaussianNoise>0.005</gaussianNoise>
+           <alwaysOn>true</alwaysOn>
+           <updateRate>50</updateRate>
+           <topicName>/${name}_ultrasonic</topicName>
+           <frameName>${name}_ultrasonic</frameName>
+           <visualize>true</visualize>
+           <radiation>ultrasonic</radiation>
+           <fov>0.261799</fov>
+        </plugin>
+     </sensor>
+   </gazebo>
+  </xacro:macro>
 </robot>

File: apollo_description/urdf/xacro/final_robot.urdf.xacro (robot description, xacro)
@@ -5,7 +5,7 @@
   <link name="base_link">
     <inertial>
-      <origin xyz="0.02 0.0 0.06" rpy="0 0 0"/>
-      <mass value="8.40"/>
-      <inertia ixx="0.10" ixy="0" ixz="0.01" iyy="0.21" iyz="0" izz="0.25"/>
+      <origin xyz="0.0 0.0 0.0" rpy="0 0 0"/>
+      <mass value="20.0"/>
+      <inertia ixx="0.16544" ixy="0" ixz="0.0" iyy="0.42368" iyz="0" izz="0.5582"/>
     </inertial>
       <visual>
@@ -22,4 +22,5 @@
       </collision>
   </link>
+  <xacro:ultrasonic name="rear" xyz="${-0.49492/2-0.05} 0 0" rpy="0 0 ${radians(180)}"/>
   <xacro:wheel wheel="fl" x_dir="0.14034" y_dir="0.1185"/>
   <xacro:wheel wheel="fr" x_dir="0.14034" y_dir="-0.1185"/>
@@ -42,10 +43,10 @@
       <odometryTopic>odom</odometryTopic>
       <odometryFrame>odom</odometryFrame>
-      <odometryRate>25.0</odometryRate>
+      <odometryRate>50.0</odometryRate>
       <robotBaseFrame>base_link</robotBaseFrame>
       <cmdVelTimeOut>0.25</cmdVelTimeOut>
       <!-- Don't publish a transform: the controller does it. -->
       <publishOdometryTf>0</publishOdometryTf>
-      <yaw_velocity_p_gain>500.0</yaw_velocity_p_gain>
+      <yaw_velocity_p_gain>50.0</yaw_velocity_p_gain>
       <x_velocity_p_gain>100.0</x_velocity_p_gain>
       <y_velocity_p_gain>100.0</y_velocity_p_gain>
@@ -53,17 +54,17 @@
     <plugin name="imu_controller" filename="libhector_gazebo_ros_imu.so">
       <robotNamespace>/</robotNamespace>
-      <updateRate>100.0</updateRate>
+      <updateRate>50.0</updateRate>
       <bodyName>imu_link</bodyName>
       <topicName>imu/data_raw</topicName>
       <accelDrift>0.0 0.0 0.0</accelDrift>
-      <accelGaussianNoise>1e-5 1e-5 1e-5</accelGaussianNoise>
-      <rateDrift>0.0000005 0.0000005 0.0000005 </rateDrift>
-      <rateGaussianNoise>0.0000001 0.0000001 0.0000001 </rateGaussianNoise>
+      <accelGaussianNoise>0.0001 0.0001 0</accelGaussianNoise>
+      <rateDrift>0.0 0.0 0.0</rateDrift>
+      <rateGaussianNoise>1e-10 1e-10 1e-10</rateGaussianNoise>
       <headingDrift>0.0</headingDrift>
-      <headingGaussianNoise>1e-8</headingGaussianNoise>
+      <headingGaussianNoise>1e-10</headingGaussianNoise>
     </plugin>
     <plugin name="mag_controller" filename="libhector_gazebo_ros_magnetic.so">
       <robotNamespace>/</robotNamespace>
-      <updateRate>100.0</updateRate>
+      <updateRate>50.0</updateRate>
       <bodyName>imu_link</bodyName>
       <topicName>imu/mag_raw</topicName>

Commit message: Indoor_localization

File: apollo_description/urdf/xacro/accessories.urdf.xacro (robot description, xacro)
@@ -97,5 +97,5 @@
            <range>
               <min>0.02</min>
-              <max>4.0</max>
+              <max>2.0</max>
               <resolution>0.02</resolution>
            </range>

File: apollo_description/urdf/xacro/final_robot.urdf.xacro (robot description, xacro)
@@ -22,5 +22,6 @@
       </collision>
   </link>
-  <xacro:ultrasonic name="rear" xyz="${-0.49492/2-0.05} 0 0" rpy="0 0 ${radians(180)}"/>
+  <xacro:ultrasonic name="rear" xyz="${-0.49492/2} 0 0" rpy="0 0 ${radians(180)}"/>
+  <xacro:ultrasonic name="front" xyz="${0.49492/2} 0 0" rpy="0 0 0"/>
   <xacro:wheel wheel="fl" x_dir="0.14034" y_dir="0.1185"/>
   <xacro:wheel wheel="fr" x_dir="0.14034" y_dir="-0.1185"/>
@@ -30,5 +31,5 @@
   <link name="imu_link"/>
   <joint name="imu_joint" type="fixed">
-    <origin xyz="0.0 0.0 0.0" rpy="0.0 0.0 0.0"/>
+    <origin xyz="0.0 0.0 0.0" rpy="0.0 0.0 ${radians(0.0)}"/>
     <parent link="base_link"/>
     <child link="imu_link"/>
@@ -48,7 +49,7 @@
       <!-- Don't publish a transform: the controller does it. -->
       <publishOdometryTf>0</publishOdometryTf>
-      <yaw_velocity_p_gain>50.0</yaw_velocity_p_gain>
-      <x_velocity_p_gain>100.0</x_velocity_p_gain>
-      <y_velocity_p_gain>100.0</y_velocity_p_gain>
+      <yaw_velocity_p_gain>500.0</yaw_velocity_p_gain>
+      <x_velocity_p_gain>10000.0</x_velocity_p_gain>
+      <y_velocity_p_gain>10000.0</y_velocity_p_gain>
     </plugin>
     <plugin name="imu_controller" filename="libhector_gazebo_ros_imu.so">
@@ -58,7 +59,7 @@
       <topicName>imu/data_raw</topicName>
       <accelDrift>0.0 0.0 0.0</accelDrift>
-      <accelGaussianNoise>0.0001 0.0001 0</accelGaussianNoise>
+      <accelGaussianNoise>1e-5 1e-5 0.0</accelGaussianNoise>
       <rateDrift>0.0 0.0 0.0</rateDrift>
-      <rateGaussianNoise>1e-10 1e-10 1e-10</rateGaussianNoise>
+      <rateGaussianNoise>1e-9 1e-9 1e-9</rateGaussianNoise>
       <headingDrift>0.0</headingDrift>
       <headingGaussianNoise>1e-10</headingGaussianNoise>

Commit message: 5ra

File: apollo_description/urdf/xacro/accessories.urdf.xacro (robot description, xacro)
@@ -1,2 +1,3 @@
+<?xml version="1.0"?>
 <robot xmlns:xacro="http://wiki.ros.org/xacro" name="kinect">
   <xacro:macro name="kinect" >
@@ -114,3 +115,82 @@
    </gazebo>
   </xacro:macro>
+  <xacro:macro name="fork_base">
+    <link name= "fork_b">
+      <visual>
+        <origin xyz="0.0 0.0 0.0" rpy="0 0 0"/>
+        <geometry>
+          <mesh filename="package://apollo_description/meshfiles/lift_base_link.STL"/>
+        </geometry>
+      </visual>
+      <inertial>
+        <origin xyz="0 0 0.0" rpy="0 0 0" />
+        <mass value="0.556" />
+        <inertia ixx="0" ixy="0" ixz="0" iyy="0" iyz="0" izz="0" />
+      </inertial>
+      <collision>
+        <geometry>
+          <box size="0.040 0.25 0.002"/>
+        </geometry>
+        <origin xyz="0.015 0 0.395"/>
+      </collision>
+    </link>
+    <joint name="base_fork_joint" type="fixed">
+      <origin xyz="-0.0250 0.0 0.0" rpy="0 0 0" />
+      <parent link="base_link" />
+      <child link="fork_b" />
+      <axis xyz="0 0 0" />
+    </joint>
+    <link name= "fork">
+      <visual>
+        <origin xyz="0.0 0.0 0.0" rpy="0 0 -1.5708"/>
+        <geometry>
+          <mesh filename="package://apollo_description/meshfiles/fork_link.STL"/>
+        </geometry>
+        <material name="fork">
+       <color rgba="0.2 1.0 1.0 1.0"/>
+     </material>
+      </visual>
+      <inertial>
+        <origin xyz="0 0 0.0" rpy="0 0 0" />
+        <mass value="0.556" />
+        <inertia ixx="0" ixy="0" ixz="0" iyy="0" iyz="0" izz="0" />
+      </inertial>
+      <collision>
+        <geometry>
+          <mesh filename="package://apollo_description/meshfiles/fork_collider.stl"/>
+        </geometry>
+        <origin xyz="0.0 0.0 0.0" rpy="0 0 -1.5708"/>
+      </collision>
+    </link>
+    <joint name="fork_joint" type="prismatic">
+      <origin xyz="0.022 0.120 0.097" rpy="0 0 0" />
+      <parent link="fork_b" />
+      <child link="fork" />
+      <axis xyz="0 0 1" />
+      <limit effort="100" velocity="0.05" lower="0.0" upper="0.275" />
+    </joint>
+    <transmission name="fork_trans">
+      <type>transmission_interface/SimpleTransmission</type>
+      <joint name="fork_joint">
+        <hardwareInterface>EffortJointInterface</hardwareInterface>
+      </joint>
+      <actuator name="fork_motor">
+        <mechanicalReduction>1</mechanicalReduction>
+        <hardwareInterface>EffortJointInterface</hardwareInterface>
+      </actuator>
+    </transmission>
+    <gazebo reference="fork">
+      <turnGravityOff>true</turnGravityOff>
+      <collision name="fork_collision">
+      <surface>
+        <friction>
+          <ode>
+            <mu>0.55</mu>
+            <mu2>0.45</mu2>
+          </ode>
+        </friction>
+      </surface>
+    </collision>
+    </gazebo>
+  </xacro:macro>
 </robot>

File: apollo_description/urdf/xacro/final_robot.urdf.xacro (robot description, xacro)
@@ -29,4 +29,5 @@
   <xacro:wheel wheel="rr" x_dir="-0.14034" y_dir="-0.1185"/>
   <xacro:kinect/>
+  <xacro:fork_base/>
   <link name="imu_link"/>
   <joint name="imu_joint" type="fixed">
