Commit message: Cleaning Up
We cleaned up the code a little.

File: apollo_description/urdf/accessories.urdf.xacro (robot description, xacro)
@@ -6,5 +6,5 @@
         <origin xyz="0 0 0" rpy="0 0 ${pi/2}"/>
         <geometry>
-          <mesh filename="package://husky_description/meshes/accessories/kinect.dae"/>
+          <mesh filename="package://apollo_description/meshes/accessories/kinect.dae"/>
         </geometry>
       </visual>
@@ -120,5 +120,5 @@
         <origin xyz="0.0 0.0 0.0" rpy="0 0 0"/>
         <geometry>
-          <mesh filename="package://apollo_description/meshfiles/lift_base_link.STL"/>
+          <mesh filename="package://apollo_description/meshes/accessories/lift_base_link.stl"/>
         </geometry>
       </visual>
@@ -145,5 +145,5 @@
         <origin xyz="0.0 0.0 0.0" rpy="0 0 -1.5708"/>
         <geometry>
-          <mesh filename="package://apollo_description/meshfiles/fork_link.STL"/>
+          <mesh filename="package://apollo_description/meshes/accessories/fork_link.stl"/>
         </geometry>
         <material name="fork">
@@ -153,10 +153,10 @@
       <inertial>
         <origin xyz="0 0 0.0" rpy="0 0 0" />
-        <mass value="0.556" />
-        <inertia ixx="0" ixy="0" ixz="0" iyy="0" iyz="0" izz="0" />
+        <mass value="1" />
+        <inertia ixx="0.166667" ixy="0" ixz="0" iyy="0.166667" iyz="0" izz="0.166667" />
       </inertial>
       <collision>
         <geometry>
-          <mesh filename="package://apollo_description/meshfiles/fork_collider.stl"/>
+          <mesh filename="package://apollo_description/meshes/accessories/fork_collider.stl"/>
         </geometry>
         <origin xyz="0.0 0.0 0.0" rpy="0 0 -1.5708"/>
@@ -170,12 +170,12 @@
       <limit effort="100" velocity="0.05" lower="0.0" upper="0.275" />
     </joint>
-    <transmission name="fork_trans">
+    <transmission name="fork_transmission">
       <type>transmission_interface/SimpleTransmission</type>
       <joint name="fork_joint">
-        <hardwareInterface>EffortJointInterface</hardwareInterface>
+        <hardwareInterface>hardware_interface/EffortJointInterface</hardwareInterface>
       </joint>
       <actuator name="fork_motor">
         <mechanicalReduction>1</mechanicalReduction>
-        <hardwareInterface>EffortJointInterface</hardwareInterface>
+        <hardwareInterface>hardware_interface/EffortJointInterface</hardwareInterface>
       </actuator>
     </transmission>
@@ -183,13 +183,51 @@
       <turnGravityOff>true</turnGravityOff>
       <collision name="fork_collision">
-      <surface>
-        <friction>
-          <ode>
-            <mu>0.55</mu>
-            <mu2>0.45</mu2>
-          </ode>
-        </friction>
-      </surface>
+        <surface>
+          <friction>
+            <ode>
+              <mu>100000</mu>
+              <mu2>100000</mu2>
+              <fdir1>0.5 0.5 0.5</fdir1>
+              <slip1>0</slip1>
+              <slip2>0</slip2>
+            </ode>
+            <torsional>
+              <coefficient>1</coefficient>
+              <patch_radius>0</patch_radius>
+              <surface_radius>0</surface_radius>
+              <use_patch_radius>1</use_patch_radius>
+              <ode>
+                <slip>0</slip>
+              </ode>
+            </torsional>
+          </friction>
+          <bounce>
+            <restitution_coefficient>0</restitution_coefficient>
+            <threshold>1e+06</threshold>
+          </bounce>
+          <contact>
+            <collide_without_contact>0</collide_without_contact>
+            <collide_without_contact_bitmask>1</collide_without_contact_bitmask>
+            <collide_bitmask>1</collide_bitmask>
+            <ode>
+              <soft_cfm>0</soft_cfm>
+              <soft_erp>0.2</soft_erp>
+              <kp>1e+13</kp>
+              <kd>1</kd>
+              <max_vel>0.01</max_vel>
+              <min_depth>0.03</min_depth>
+            </ode>
+            <bullet>
+              <split_impulse>1</split_impulse>
+              <split_impulse_penetration_threshold>-0.01</split_impulse_penetration_threshold>
+              <soft_cfm>0</soft_cfm>
+              <soft_erp>0.2</soft_erp>
+              <kp>1e+13</kp>
+              <kd>1</kd>
+            </bullet>
+          </contact>
+        </surface>
     </collision>
+    <implicitSpringDamper>1</implicitSpringDamper>
     </gazebo>
   </xacro:macro>

File: apollo_description/urdf/apollo.urdf.xacro (robot description, xacro)
@@ -1,6 +1,6 @@
 <?xml version="1.0"?>
 <robot xmlns:xacro="http://wiki.ros.org/xacro" name="apollo">
-  <xacro:include filename="$(find apollo_description)/urdf/xacro/wheel.urdf.xacro"/>
-  <xacro:include filename="$(find apollo_description)/urdf/xacro/accessories.urdf.xacro"/>
+  <xacro:include filename="$(find apollo_description)/urdf/wheel.urdf.xacro"/>
+  <xacro:include filename="$(find apollo_description)/urdf/accessories.urdf.xacro"/>
   <link name="base_link">
     <inertial>
@@ -11,5 +11,5 @@
       <visual>
           <geometry>
-            <mesh filename="package://apollo_description/meshfiles/base_link.STL"/>
+            <mesh filename="package://apollo_description/meshes/base_link.stl"/>
           </geometry>
           <origin xyz="0 0 0"/>

File: apollo_description/urdf/wheel.urdf.xacro (robot description, xacro)
@@ -10,5 +10,5 @@
       <visual>
           <geometry>
-              <mesh filename="package://apollo_description/meshfiles/wheel.stl"/>
+              <mesh filename="package://apollo_description/meshes/wheel.stl"/>
           </geometry>
           <origin xyz ="0 0 0" rpy ="0 0 1.5707963268"/>

Commit message: added base

File: apollo_description/urdf/accessories.urdf.xacro (robot description, xacro)
@@ -173,9 +173,9 @@
       <type>transmission_interface/SimpleTransmission</type>
       <joint name="fork_joint">
-        <hardwareInterface>hardware_interface/EffortJointInterface</hardwareInterface>
+        <hardwareInterface>hardware_interface/PositionJointInterface</hardwareInterface>
       </joint>
       <actuator name="fork_motor">
         <mechanicalReduction>1</mechanicalReduction>
-        <hardwareInterface>hardware_interface/EffortJointInterface</hardwareInterface>
+        <hardwareInterface>hardware_interface/PositionJointInterface</hardwareInterface>
       </actuator>
     </transmission>

File: apollo_description/urdf/apollo.urdf.xacro (robot description, xacro)
@@ -4,9 +4,4 @@
   <xacro:include filename="$(find apollo_description)/urdf/accessories.urdf.xacro"/>
   <link name="base_link">
-    <inertial>
-      <origin xyz="0.0 0.0 0.0" rpy="0 0 0"/>
-      <mass value="20.0"/>
-      <inertia ixx="0.16544" ixy="0" ixz="0.0" iyy="0.42368" iyz="0" izz="0.5582"/>
-    </inertial>
       <visual>
           <geometry>
@@ -22,4 +17,15 @@
       </collision>
   </link>
+  <link name="inertial_link">
+    <inertial>
+      <origin xyz="0.0 0.0 0.0" rpy="0 0 0"/>
+      <mass value="20.0"/>
+      <inertia ixx="0.16544" ixy="0" ixz="0.0" iyy="0.42368" iyz="0" izz="0.5582"/>
+    </inertial>
+  </link>
+  <joint name="inertial" type="fixed">
+    <parent link="base_link"/>
+    <child link="inertial_link"/>
+  </joint>
   <xacro:ultrasonic name="rear" xyz="${-0.49492/2} 0 0" rpy="0 0 ${radians(180)}"/>
   <xacro:ultrasonic name="front" xyz="${0.49492/2} 0 0" rpy="0 0 0"/>
